File: mcu.kicad_sch (KiCad schematic)
At the start: 33 parts, among them J2 GSD090012SEU, Q2 BC817, Q3 BC817, SW1 Boot, SW2 Reset, U3 ESP32-C3-WROOM-02, U4 CP2102N-A02-GQFN20, U5 USBLC6-2SC6, U6 W25Q32JVSSIQ

Commit message: components arranged
Parts:
- removed C24: 0.1u, symbol Device:C
- removed SW1: Boot, Button_Switch_SMD:Nidec_Copal_CAS-120A, symbol Switch:SW_Nidec_CAS-120A1
- removed SW2: Reset, Button_Switch_SMD:Nidec_Copal_CAS-120A, symbol Switch:SW_Nidec_CAS-120A1
- added C26: 0.1u, Capacitor_SMD:C_0805_2012Metric, symbol Device:C
- added J3: Conn_01x05_Pin, Connector_PinHeader_2.54mm:PinHeader_1x05_P2.54mm_Vertical_SMD_Pin1Left, symbol Connector:Conn_01x05_Pin
- added SW3, SW4: SW_MEC_5E, USLPT2819DT2TR:SW_USLPT2819DT2TR, symbol Switch:SW_MEC_5E
- C10, C11, C12, C13, C14, C25, C7, C8, C9: footprint (none) -> Capacitor_SMD:C_0805_2012Metric
- D5, D6: footprint (none) -> LED_SMD:LED_1206_3216Metric
- R10, R11, R12, R13, R14, R15, R16, R17, R18, R19, R30, R31: footprint (none) -> Resistor_SMD:R_0805_2012Metric
Connections:
- net +3v3: now also C7.1, J3.1 (Pin_1); no longer C7.2
- net BOOT: now also U3.8 (IO9), C26.2, SW4.3 (K), SW4.4 (A)
- net EN: now also C25.2, SW3.3 (K), SW3.4 (A); no longer C25.1
- net GND: now also C25.1, C7.2, U5.2 (GND), C26.1, J3.5 (Pin_5), SW3.1, SW3.2, SW4.1, SW4.2; no longer C25.2, C7.1
- net GPIO18: now reaches U3.13 (IO18)
- net GPIO18: now also J3.3 (Pin_3)
- net GPIO19: now reaches U3.14 (IO19)
- net GPIO19: now also J3.4 (Pin_4)
- net SCL: now reaches U3.15 (IO3)
- net PHOTO: now reaches U3.17 (IO1)
- net MIC_OUT: now reaches U3.18 (IO0)
- net SDA: now reaches U3.3 (IO4)
- net GPIO8: now reaches U3.7 (IO8)
- net GPIO8: now also J3.2 (Pin_2)
Other:
- moved on the sheet: C25, C7, Q2, Q3, R30, R31

Commit message: complete pcb
Parts:
- added H1, H2, H3, H4: MountingHole, MountingHole:MountingHole_2.2mm_M2_DIN965_Pad_TopBottom, symbol Mechanical:MountingHole
Connections:
- net CTS is gone; now on net DTR: U4.15 (CTS)
- net VBUS: now also C11.2, R11.2, R12.1, U4.8 (VBUS)
