File: sensor-board.kicad_pcb (KiCad board)
At the start: 2 copper layers, 5 x 8.2 mm, 82 parts, among them J1 Conn_01x02_Pin, J2 GSD090012SEU, J3 Conn_01x05_Pin, P1 USB_C_Plug_USB2.0, Q1 TEMT6000X01, Q2 BC817, Q3 BC817, SW3 SW_MEC_5E, SW4 SW_MEC_5E, U1 MCP73871, U2 LM1117DT-3.3, U3 ESP32-C3-WROOM-02, U4 CP2102N-A02-GQFN20, U5 USBLC6-2SC6, U6 W25Q32JVSSIQ, U7 BME280, U8 MAX4466EXK

Commit message: complete pcb
Parts:
- added H1: MountingHole, MountingHole:MountingHole_2.2mm_M2_DIN965_Pad_TopBottom, F.Cu at (122.1, 85.3)
- added H2: MountingHole, MountingHole:MountingHole_2.2mm_M2_DIN965_Pad_TopBottom, F.Cu at (122.1, 122.8)
- added H3: MountingHole, MountingHole:MountingHole_2.2mm_M2_DIN965_Pad_TopBottom, F.Cu at (200.8, 85.3)
- added H4: MountingHole, MountingHole:MountingHole_2.2mm_M2_DIN965_Pad_TopBottom, F.Cu at (200.8, 122.8)
- J1: moved to B.Cu
- P1: footprint Connector_USB:USB_C_Plug_JAE_DX07P024AJ1 -> Connector_USB:USB_C_Receptacle_Amphenol_124019772112A
- moved R9 124.8 mm to (138.8, 98.8), turned to 90 degrees
- moved D4 117.6 mm to (137.3, 95.2), turned to 180 degrees
- moved U5 107.5 mm to (154.4, 105.3), turned to -90 degrees
- moved C10 106.8 mm to (157.4, 105.3), turned to -90 degrees
- moved D5 105.8 mm to (144.1, 107.4), turned to 180 degrees
- moved R13 105.6 mm to (148.4, 107.5), turned to 180 degrees
- moved D2 104.3 mm to (139.1, 109.2), turned to -90 degrees
- moved D3 102.5 mm to (136.2, 109.2), turned to -90 degrees
- moved C9 102.5 mm to (159.3, 101.3), turned to 180 degrees
- moved D6 101.1 mm to (144.1, 104.0), turned to 180 degrees
- moved R14 100.8 mm to (148.4, 104.1), turned to 180 degrees
- moved D1 100.7 mm to (133.3, 109.3), turned to -90 degrees
- moved U4 100.4 mm to (155.2, 100.2), turned to 90 degrees
- moved R10 99.6 mm to (159.3, 99.0), turned to 180 degrees
- moved R7 99.0 mm to (139.1, 104.8), turned to 90 degrees
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Connections:
- C11 pad 2: Net-(C11-Pad2) -> VBUS
- R11 pad 2: Net-(C11-Pad2) -> VBUS
- R12 pad 1: Net-(C11-Pad2) -> VBUS
- U4 pad 15: CTS -> DTR
- U4 pad 8: unconnected-(U4-VBUS-Pad8) -> VBUS
Routing:
- net VBUS: track 0.00 -> 79.9 mm, vias 0 -> 4
- net +3v3: track 0.00 -> 66.9 mm, vias 0 -> 19
- net SCLK: track 0.00 -> 50.5 mm, vias 0 -> 4
- net GND: track 0.00 -> 49.6 mm, vias 0 -> 13
- net MIC_OUT: track 0.00 -> 46.1 mm, vias 0 -> 2
- net GPIO8: track 0.00 -> 46.0 mm, vias 0 -> 2
- net D-: track 0.00 -> 39.4 mm, vias 0 -> 4
- net MOSI_DI: track 0.00 -> 36.8 mm, vias 0 -> 2
- net MISO_DO: track 0.00 -> 36.5 mm, vias 0 -> 4
- net DTR: track 0.00 -> 36.2 mm, vias 0 -> 2
- net D+: track 0.00 -> 36.1 mm, vias 0 -> 2
- net CS_SD: track 0.00 -> 35.9 mm, vias 0 -> 2
- net SDA: track 0.00 -> 32.8 mm, vias 0 -> 4
- net RTS: track 0.00 -> 31.6 mm, vias 0 -> 2
- net SCL: track 0.00 -> 29.0 mm, vias 0 -> 2
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- added copper zone on B.Cu, net +3v3
- added copper zone on F.Cu, net GND
Other:
- board size 5 x 8.2 mm -> 86.8 x 45.5 mm
